File: schem/main_schem/power.sch (KiCad schematic (older format))
At the start: 0 parts

Commit message: linear regulators for logic/mcu
Parts:
- added C?: 0.1uF, symbol CP
- added C?: 0.33uF, symbol CP
- added C?: 10uF, symbol CP
- added U?: LM7805, symbol LM7805
- added U?: LM1117-3.3, symbol LM7805
Connections:
- new net +24V: C?.1, U?.VI
- new net +3.3V: C?.1, U?.VO
- new net +5V: C?.1, U?.VI, U?.VO
- new net GND: C?.2, C?.2, C?.2, U?.GND, U?.GND
Other:
- note added: "DIGITAL SYSTEM REGULATORS"
- note added: "These grounds should be connected via single points only,\n possibly with ferrite beads between them to minimize transients."
Changed lines of the file:
@@
-EESchema Schematic File Version 2  date 9/29/2012 1:33:09 PM
+EESchema Schematic File Version 2  date 9/29/2012 2:30:36 PM
 LIBS:power
 LIBS:device
@@
 Comment4 ""
 $EndDescr
+Text Notes 9700 800  0    30   ~ 0
+These grounds should be connected via single points only,\n possibly with ferrite beads between them to minimize transients.
+Connection ~ 10250 900
+Wire Wire Line
+	10650 900  10650 1000
+Wire Wire Line
+	10650 900  9850 900
+Wire Notes Line
+	11150 2350 6350 2350
+Wire Notes Line
+	6350 2350 6350 500
+Wire Wire Line
+	6700 1100 6700 1350
+Wire Wire Line
+	8050 1800 8050 2050
+Connection ~ 9350 1350
+Wire Wire Line
+	6900 1800 6900 2050
+Wire Wire Line
+	7450 1650 7450 2050
+Connection ~ 8150 1350
+Wire Wire Line
+	8150 1100 8150 1350
+Wire Wire Line
+	6700 1350 7050 1350
+Wire Wire Line
+	7850 1350 8400 1350
+Wire Wire Line
+	8050 1400 8050 1350
+Connection ~ 8050 1350
+Wire Wire Line
+	6900 1400 6900 1350
+Connection ~ 6900 1350
+Wire Wire Line
+	9200 1350 9450 1350
+Wire Wire Line
+	9450 1350 9450 1400
+Wire Wire Line
+	8800 1650 8800 2050
+Wire Wire Line
+	9350 1100 9350 1350
+Wire Wire Line
+	9450 1800 9450 2050
+Wire Wire Line
+	9850 900  9850 1000
+Wire Wire Line
+	10250 900  10250 1000
+$Comp
+L GNDPWR #PWR?
+U 1 1 50674BFE
+P 10650 1000
+F 0 "#PWR?" H 10650 1050 40  0001 C CNN
+F 1 "GNDPWR" H 10650 920 40  0000 C CNN
+	1    10650 1000
+	1    0    0    -1
+$EndComp
+$Comp
+L VSS #PWR?
+U 1 1 50674BEC
+P 10250 1000
+F 0 "#PWR?" H 10250 1000 30  0001 C CNN
+F 1 "VSS" H 10250 930 30  0000 C CNN
+	1    10250 1000
+	1    0    0    -1
+$EndComp
+$Comp
+L GND #PWR?
+U 1 1 50674BE7
+P 9850 1000
+F 0 "#PWR?" H 9850 1000 30  0001 C CNN
+F 1 "GND" H 9850 930 30  0001 C CNN
+	1    9850 1000
+	1    0    0    -1
+$EndComp
+Text Notes 6600 650  0    60   ~ 0
+DIGITAL SYSTEM REGULATORS
+$Comp
+L GND #PWR?
+U 1 1 50674B55
+P 9450 2050
+F 0 "#PWR?" H 9450 2050 30  0001 C CNN
+F 1 "GND" H 9450 1980 30  0001 C CNN
+	1    9450 2050
+	1    0    0    -1
+$EndComp
+$Comp
+L GND #PWR?
+U 1 1 50674B26
+P 8050 2050
+F 0 "#PWR?" H 8050 2050 30  0001 C CNN
+F 1 "GND" H 8050 1980 30  0001 C CNN
+	1    8050 2050
+	1    0    0    -1
+$EndComp
+$Comp
+L GND #PWR?
+U 1 1 50674B1A
+P 8800 2050
+F 0 "#PWR?" H 8800 2050 30  0001 C CNN
+F 1 "GND" H 8800 1980 30  0001 C CNN
+	1    8800 2050
+	1    0    0    -1
+$EndComp
+$Comp
+L +3.3V #PWR?
+U 1 1 50674AF6
+P 9350 1100
+F 0 "#PWR?" H 9350 1060 30  0001 C CNN
+F 1 "+3.3V" H 9350 1210 30  0000 C CNN
+	1    9350 1100
+	1    0    0    -1
+$EndComp
+$Comp
+L GNDPWR #PWR?
+U 1 1 506749D8
+P 6900 2050
+F 0 "#PWR?" H 6900 2100 40  0001 C CNN
+F 1 "GNDPWR" H 6900 1970 40  0000 C CNN
+	1    6900 2050
+	1    0    0    -1
+$EndComp
+$Comp
+L CP C?
+U 1 1 506749BB
+P 9450 1600
+F 0 "C?" H 9500 1700 50  0000 L CNN
+F 1 "10uF" H 9500 1500 50  0000 L CNN
+	1    9450 1600
+	1    0    0    -1
+$EndComp
+$Comp
+L CP C?
+U 1 1 506749B5
+P 6900 1600
+F 0 "C?" H 6950 1700 50  0000 L CNN
+F 1 "0.33uF" H 6950 1500 50  0000 L CNN
+	1    6900 1600
+	1    0    0    -1
+$EndComp
+$Comp
+L GNDPWR #PWR?
+U 1 1 506749A3
+P 7450 2050
+F 0 "#PWR?" H 7450 2100 40  0001 C CNN
+F 1 "GNDPWR" H 7450 1970 40  0000 C CNN
+	1    7450 2050
+	1    0    0    -1
+$EndComp
+$Comp
+L CP C?
+U 1 1 50674985
+P 8050 1600
+F 0 "C?" H 8100 1700 50  0000 L CNN
+F 1 "0.1uF" H 8100 1500 50  0000 L CNN
+	1    8050 1600
+	1    0    0    -1
+$EndComp
+$Comp
+L +5V #PWR?
+U 1 1 50674976
+P 8150 1100
+F 0 "#PWR?" H 8150 1190 20  0001 C CNN
+F 1 "+5V" H 8150 1190 30  0000 C CNN
+	1    8150 1100
+	1    0    0    -1
+$EndComp
+$Comp
+L +24V #PWR?
+U 1 1 50674960
+P 6700 1100
+F 0 "#PWR?" H 6700 1050 20  0001 C CNN
+F 1 "+24V" H 6700 1200 30  0000 C CNN
+	1    6700 1100
+	1    0    0    -1
+$EndComp
+$Comp
+L LM7805 U?
+U 1 1 50674945
+P 8800 1400
+F 0 "U?" H 8950 1204 60  0000 C CNN
+F 1 "LM1117-3.3" H 8800 1600 60  0000 C CNN
+	1    8800 1400
+	1    0    0    -1
+$EndComp
+$Comp
+L LM7805 U?
+U 1 1 5067487E
+P 7450 1400
+F 0 "U?" H 7600 1204 60  0000 C CNN
+F 1 "LM7805" H 7450 1600 60  0000 C CNN
+	1    7450 1400
+	1    0    0    -1
+$EndComp
 $EndSCHEMATC
