File: schem/main_schem/power.sch (KiCad schematic (older format))
At the start: 5 parts

Commit message: Begin board, layout mcu, xtal, eeprom
Parts:
- gave numbers to parts that had none: 5
Changed lines of the file:
@@
-EESchema Schematic File Version 2  date 9/29/2012 4:29:19 PM
+EESchema Schematic File Version 2  date 10/1/2012 7:44:23 AM
 LIBS:power
 LIBS:device
@@
 $Descr A4 11700 8267
 encoding utf-8
-Sheet 4 6
+Sheet 4 5
 Title "Power Subsystem"
-Date "29 sep 2012"
+Date "1 oct 2012"
 Rev ""
 Comp "Ingersoll Rand 402 Senior Design group."
@@
 Connection ~ 10250 900
 Wire Wire Line
-	10650 900  10650 1000
+	10650 1000 10650 900
 Wire Wire Line
 	10650 900  9850 900
@@
 	10250 900  10250 1000
 $Comp
-L GNDPWR #PWR?
+L GNDPWR #PWR045
 U 1 1 50674BFE
 P 10650 1000
-F 0 "#PWR?" H 10650 1050 40  0001 C CNN
+F 0 "#PWR045" H 10650 1050 40  0001 C CNN
 F 1 "GNDPWR" H 10650 920 40  0000 C CNN
 	1    10650 1000
@@
 $EndComp
 $Comp
-L VSS #PWR?
+L VSS #PWR046
 U 1 1 50674BEC
 P 10250 1000
-F 0 "#PWR?" H 10250 1000 30  0001 C CNN
+F 0 "#PWR046" H 10250 1000 30  0001 C CNN
 F 1 "VSS" H 10250 930 30  0000 C CNN
 	1    10250 1000
@@
 $EndComp
 $Comp
-L GND #PWR?
+L GND #PWR047
 U 1 1 50674BE7
 P 9850 1000
-F 0 "#PWR?" H 9850 1000 30  0001 C CNN
+F 0 "#PWR047" H 9850 1000 30  0001 C CNN
 F 1 "GND" H 9850 930 30  0001 C CNN
 	1    9850 1000
@@
 DIGITAL SYSTEM REGULATORS
 $Comp
-L GND #PWR?
+L GND #PWR048
 U 1 1 50674B55
 P 9450 2050
-F 0 "#PWR?" H 9450 2050 30  0001 C CNN
+F 0 "#PWR048" H 9450 2050 30  0001 C CNN
 F 1 "GND" H 9450 1980 30  0001 C CNN
 	1    9450 2050
@@
 $EndComp
 $Comp
-L GND #PWR?
+L GND #PWR049
 U 1 1 50674B26
 P 8050 2050
-F 0 "#PWR?" H 8050 2050 30  0001 C CNN
+F 0 "#PWR049" H 8050 2050 30  0001 C CNN
 F 1 "GND" H 8050 1980 30  0001 C CNN
 	1    8050 2050
@@
 $EndComp
 $Comp
-L GND #PWR?
+L GND #PWR050
 U 1 1 50674B1A
 P 8800 2050
-F 0 "#PWR?" H 8800 2050 30  0001 C CNN
+F 0 "#PWR050" H 8800 2050 30  0001 C CNN
 F 1 "GND" H 8800 1980 30  0001 C CNN
 	1    8800 2050
@@
 $EndComp
 $Comp
-L +3.3V #PWR?
+L +3.3V #PWR051
 U 1 1 50674AF6
 P 9350 1100
-F 0 "#PWR?" H 9350 1060 30  0001 C CNN
+F 0 "#PWR051" H 9350 1060 30  0001 C CNN
 F 1 "+3.3V" H 9350 1210 30  0000 C CNN
 	1    9350 1100
@@
 $EndComp
 $Comp
-L GNDPWR #PWR?
+L GNDPWR #PWR052
 U 1 1 506749D8
 P 6900 2050
-F 0 "#PWR?" H 6900 2100 40  0001 C CNN
+F 0 "#PWR052" H 6900 2100 40  0001 C CNN
 F 1 "GNDPWR" H 6900 1970 40  0000 C CNN
 	1    6900 2050
@@
 $EndComp
 $Comp
-L CP C?
+L CP C19
 U 1 1 506749BB
 P 9450 1600
-F 0 "C?" H 9500 1700 50  0000 L CNN
+F 0 "C19" H 9500 1700 50  0000 L CNN
 F 1 "10uF" H 9500 1500 50  0000 L CNN
 	1    9450 1600
@@
 $EndComp
 $Comp
-L CP C?
+L CP C17
 U 1 1 506749B5
 P 6900 1600
-F 0 "C?" H 6950 1700 50  0000 L CNN
+F 0 "C17" H 6950 1700 50  0000 L CNN
 F 1 "0.33uF" H 6950 1500 50  0000 L CNN
 	1    6900 1600
@@
 $EndComp
 $Comp
-L GNDPWR #PWR?
+L GNDPWR #PWR053
 U 1 1 506749A3
 P 7450 2050
-F 0 "#PWR?" H 7450 2100 40  0001 C CNN
+F 0 "#PWR053" H 7450 2100 40  0001 C CNN
 F 1 "GNDPWR" H 7450 1970 40  0000 C CNN
 	1    7450 2050
@@
 $EndComp
 $Comp
-L CP C?
+L CP C18
 U 1 1 50674985
 P 8050 1600
-F 0 "C?" H 8100 1700 50  0000 L CNN
+F 0 "C18" H 8100 1700 50  0000 L CNN
 F 1 "0.1uF" H 8100 1500 50  0000 L CNN
 	1    8050 1600
@@
 $EndComp
 $Comp
-L +5V #PWR?
+L +5V #PWR054
 U 1 1 50674976
 P 8150 1100
-F 0 "#PWR?" H 8150 1190 20  0001 C CNN
+F 0 "#PWR054" H 8150 1190 20  0001 C CNN
 F 1 "+5V" H 8150 1190 30  0000 C CNN
 	1    8150 1100
@@
 $EndComp
 $Comp
-L +24V #PWR?
+L +24V #PWR055
 U 1 1 50674960
 P 6700 1100
-F 0 "#PWR?" H 6700 1050 20  0001 C CNN
+F 0 "#PWR055" H 6700 1050 20  0001 C CNN
 F 1 "+24V" H 6700 1200 30  0000 C CNN
 	1    6700 1100
@@
 $EndComp
 $Comp
-L LM7805 U?
+L LM7805 U5
 U 1 1 50674945
 P 8800 1400
-F 0 "U?" H 8950 1204 60  0000 C CNN
+F 0 "U5" H 8950 1204 60  0000 C CNN
 F 1 "LM1117-3.3" H 8800 1600 60  0000 C CNN
 	1    8800 1400
@@
 $EndComp
 $Comp
-L LM7805 U?
+L LM7805 U4
 U 1 1 5067487E
 P 7450 1400
-F 0 "U?" H 7600 1204 60  0000 C CNN
+F 0 "U4" H 7600 1204 60  0000 C CNN
 F 1 "LM7805" H 7450 1600 60  0000 C CNN
 	1    7450 1400

Commit message: BOM sheets, update ethernet analog circuit
Parts:
- renumbered C17 to C19, C18 to C20, C19 to C21, U4 to U6, U5 to U7
Changed lines of the file:
@@
-EESchema Schematic File Version 2  date 10/5/2012 10:31:23 AM
+EESchema Schematic File Version 2  date 10/5/2012 11:52:46 PM
 LIBS:power
 LIBS:device
@@
 $Descr A4 11700 8267
 encoding utf-8
-Sheet 4 6
+Sheet 5 6
 Title "Power Subsystem"
-Date "5 oct 2012"
+Date "6 oct 2012"
 Rev ""
 Comp "Ingersoll Rand 402 Senior Design group."
@@
 	10250 900  10250 1000
 $Comp
-L GNDPWR #PWR045
+L GNDPWR #PWR054
 U 1 1 50674BFE
 P 10650 1000
-F 0 "#PWR045" H 10650 1050 40  0001 C CNN
+F 0 "#PWR054" H 10650 1050 40  0001 C CNN
 F 1 "GNDPWR" H 10650 920 40  0000 C CNN
 	1    10650 1000
@@
 $EndComp
 $Comp
-L VSS #PWR046
+L VSS #PWR055
 U 1 1 50674BEC
 P 10250 1000
-F 0 "#PWR046" H 10250 1000 30  0001 C CNN
+F 0 "#PWR055" H 10250 1000 30  0001 C CNN
 F 1 "VSS" H 10250 930 30  0000 C CNN
 	1    10250 1000
@@
 $EndComp
 $Comp
-L GND #PWR047
+L GND #PWR056
 U 1 1 50674BE7
 P 9850 1000
-F 0 "#PWR047" H 9850 1000 30  0001 C CNN
+F 0 "#PWR056" H 9850 1000 30  0001 C CNN
 F 1 "GND" H 9850 930 30  0001 C CNN
 	1    9850 1000
@@
 DIGITAL SYSTEM REGULATORS
 $Comp
-L GND #PWR048
+L GND #PWR057
 U 1 1 50674B55
 P 9450 2050
-F 0 "#PWR048" H 9450 2050 30  0001 C CNN
+F 0 "#PWR057" H 9450 2050 30  0001 C CNN
 F 1 "GND" H 9450 1980 30  0001 C CNN
 	1    9450 2050
@@
 $EndComp
 $Comp
-L GND #PWR049
+L GND #PWR058
 U 1 1 50674B26
 P 8050 2050
-F 0 "#PWR049" H 8050 2050 30  0001 C CNN
+F 0 "#PWR058" H 8050 2050 30  0001 C CNN
 F 1 "GND" H 8050 1980 30  0001 C CNN
 	1    8050 2050
@@
 $EndComp
 $Comp
-L GND #PWR050
+L GND #PWR059
 U 1 1 50674B1A
 P 8800 2050
-F 0 "#PWR050" H 8800 2050 30  0001 C CNN
+F 0 "#PWR059" H 8800 2050 30  0001 C CNN
 F 1 "GND" H 8800 1980 30  0001 C CNN
 	1    8800 2050
@@
 $EndComp
 $Comp
-L +3.3V #PWR051
+L +3.3V #PWR060
 U 1 1 50674AF6
 P 9350 1100
-F 0 "#PWR051" H 9350 1060 30  0001 C CNN
+F 0 "#PWR060" H 9350 1060 30  0001 C CNN
 F 1 "+3.3V" H 9350 1210 30  0000 C CNN
 	1    9350 1100
@@
 $EndComp
 $Comp
-L GNDPWR #PWR052
+L GNDPWR #PWR061
 U 1 1 506749D8
 P 6900 2050
-F 0 "#PWR052" H 6900 2100 40  0001 C CNN
+F 0 "#PWR061" H 6900 2100 40  0001 C CNN
 F 1 "GNDPWR" H 6900 1970 40  0000 C CNN
 	1    6900 2050
@@
 $EndComp
 $Comp
-L CP C19
+L CP C21
 U 1 1 506749BB
 P 9450 1600
-F 0 "C19" H 9500 1700 50  0000 L CNN
+F 0 "C21" H 9500 1700 50  0000 L CNN
 F 1 "10uF" H 9500 1500 50  0000 L CNN
 	1    9450 1600
@@
 $EndComp
 $Comp
-L CP C17
+L CP C19
 U 1 1 506749B5
 P 6900 1600
-F 0 "C17" H 6950 1700 50  0000 L CNN
+F 0 "C19" H 6950 1700 50  0000 L CNN
 F 1 "0.33uF" H 6950 1500 50  0000 L CNN
 	1    6900 1600
@@
 $EndComp
 $Comp
-L GNDPWR #PWR053
+L GNDPWR #PWR062
 U 1 1 506749A3
 P 7450 2050
-F 0 "#PWR053" H 7450 2100 40  0001 C CNN
+F 0 "#PWR062" H 7450 2100 40  0001 C CNN
 F 1 "GNDPWR" H 7450 1970 40  0000 C CNN
 	1    7450 2050
@@
 $EndComp
 $Comp
-L CP C18
+L CP C20
 U 1 1 50674985
 P 8050 1600
-F 0 "C18" H 8100 1700 50  0000 L CNN
+F 0 "C20" H 8100 1700 50  0000 L CNN
 F 1 "0.1uF" H 8100 1500 50  0000 L CNN
 	1    8050 1600
@@
 $EndComp
 $Comp
-L +5V #PWR054
+L +5V #PWR063
 U 1 1 50674976
 P 8150 1100
-F 0 "#PWR054" H 8150 1190 20  0001 C CNN
+F 0 "#PWR063" H 8150 1190 20  0001 C CNN
 F 1 "+5V" H 8150 1190 30  0000 C CNN
 	1    8150 1100
@@
 $EndComp
 $Comp
-L +24V #PWR055
+L +24V #PWR064
 U 1 1 50674960
 P 6700 1100
-F 0 "#PWR055" H 6700 1050 20  0001 C CNN
+F 0 "#PWR064" H 6700 1050 20  0001 C CNN
 F 1 "+24V" H 6700 1200 30  0000 C CNN
 	1    6700 1100
@@
 $EndComp
 $Comp
-L LM7805 U5
+L LM7805 U7
 U 1 1 50674945
 P 8800 1400
-F 0 "U5" H 8950 1204 60  0000 C CNN
+F 0 "U7" H 8950 1204 60  0000 C CNN
 F 1 "LM1117-3.3" H 8800 1600 60  0000 C CNN
 	1    8800 1400
@@
 $EndComp
 $Comp
-L LM7805 U4
+L LM7805 U6
 U 1 1 5067487E
 P 7450 1400
-F 0 "U4" H 7600 1204 60  0000 C CNN
+F 0 "U6" H 7600 1204 60  0000 C CNN
 F 1 "LM7805" H 7450 1600 60  0000 C CNN
 	1    7450 1400
