File: schem/main_schem/QEL_drive.sch (KiCad schematic (older format))
At the start: 7 parts, among them P1 CONN_2, Q1 ENHANCED_MOSFET_N, U3 PS2501-1

Commit message: Port for manually actuating QEL, update BOM
Parts:
- added P8: CONN_2, symbol CONN_2
Connections:
- net GNDPWR: now also P8.2 (PM)
- net at D1.1 (A), P1.2 (PM), Q1.D: now also P8.1 (P1)
Changed lines of the file:
@@
-EESchema Schematic File Version 2  date 10/24/2012 8:18:13 AM
+EESchema Schematic File Version 2  date 10/26/2012 9:37:13 AM
 LIBS:power
 LIBS:device
@@
 Sheet 3 6
 Title "QEL_Driver"
-Date "24 oct 2012"
+Date "26 oct 2012"
 Rev "2"
 Comp "ECE 402 Senior Design"
@@
 Comment4 ""
 $EndDescr
-$Comp
-L PS2501-1 U3
-U 1 1 5072317B
-P 5700 3550
-F 0 "U3" H 5675 3775 60  0000 C CNN
-F 1 "PS2501-1" H 5700 3250 60  0000 C CNN
-	1    5700 3550
-	1    0    0    -1
-$EndComp
+Connection ~ 8150 4350
+Wire Wire Line
+	8150 4350 8550 4350
+Wire Wire Line
+	8550 4350 8550 4150
 Wire Wire Line
 	8150 4250 8150 4550
@@
 	4850 3650 5050 3650
 Connection ~ 7700 3450
+Wire Wire Line
+	8400 3650 8400 3950
+Wire Wire Line
+	8400 3950 8550 3950
+Connection ~ 8400 3650
 $Comp
-L GNDPWR #PWR010
+L CONN_2 P8
+U 1 1 508A9634
+P 8900 4050
+F 0 "P8" V 8850 4050 40  0000 C CNN
+F 1 "CONN_2" V 8950 4050 40  0000 C CNN
+	1    8900 4050
+	1    0    0    -1
+$EndComp
+$Comp
+L PS2501-1 U3
+U 1 1 5072317B
+P 5700 3550
+F 0 "U3" H 5675 3775 60  0000 C CNN
+F 1 "PS2501-1" H 5700 3250 60  0000 C CNN
+	1    5700 3550
+	1    0    0    -1
+$EndComp
+$Comp
+L GNDPWR #PWR13
 U 1 1 506747B4
 P 8150 4550
-F 0 "#PWR010" H 8150 4600 40  0001 C CNN
+F 0 "#PWR13" H 8150 4600 40  0001 C CNN
 F 1 "GNDPWR" H 8150 4470 40  0000 C CNN
 	1    8150 4550
@@
 $EndComp
 $Comp
-L GNDPWR #PWR011
+L GNDPWR #PWR11
 U 1 1 506747A8
 P 7000 4550
-F 0 "#PWR011" H 7000 4600 40  0001 C CNN
+F 0 "#PWR11" H 7000 4600 40  0001 C CNN
 F 1 "GNDPWR" H 7000 4470 40  0000 C CNN
 	1    7000 4550
@@
 $EndComp
 $Comp
-L VSS #PWR012
+L VSS #PWR10
 U 1 1 50674779
 P 4300 3800
-F 0 "#PWR012" H 4300 3800 30  0001 C CNN
+F 0 "#PWR10" H 4300 3800 30  0001 C CNN
 F 1 "VSS" H 4300 3730 30  0000 C CNN
 	1    4300 3800
@@
 $EndComp
 $Comp
-L +24V #PWR013
+L +24V #PWR12
 U 1 1 504BA51D
 P 7250 3400
-F 0 "#PWR013" H 7250 3350 20  0001 C CNN
+F 0 "#PWR12" H 7250 3350 20  0001 C CNN
 F 1 "+24V" H 7250 3500 30  0000 C CNN
 	1    7250 3400
